Commit message: expand link names after macro calls

File: examples/generated/PiTasc/ati_axia80.xacro (robot description, xacro)
@@ -15,15 +15,15 @@
 		<joint name="${prefix}robotside_joint" type="fixed">
 			<parent link="${parent_link}" />
-			<child link="${prefix}robotside" />
+			<child link="ati_axia80_robotside" />
 			<xacro:insert_block name="origin_joint"/>
 		</joint>
 		<joint name="${prefix}toolside_joint" type="fixed">
-			<parent link="${prefix}robotside" />
-			<child link="${prefix}toolside" />
+			<parent link="ati_axia80_robotside" />
+			<child link="ati_axia80_toolside" />
 			<origin xyz="0 0 0" rpy="0 0 0.0254" />
 		</joint>
 		<joint name="${prefix}measurement_joint" type="fixed">
-			<parent link="${prefix}toolside" />
-			<child link="${prefix}force_sensor_frame" />
+			<parent link="ati_axia80_toolside" />
+			<child link="ati_axia80_force_sensor_frame" />
 			<origin xyz="0 0 0" rpy="0 0 0" />
 		</joint>

File: examples/generated/PiTasc/kr16.xacro (robot description, xacro)
@@ -4,7 +4,7 @@
 	<xacro:include filename="$(find kr16_description)/urdf/axia80_adapter_plates.xacro" />
 	<xacro:include filename="$(find kr16_description)/urdf/ati_axia80.xacro" />
-	<xacro:kuka_kr16_2  prefix="kr16">
+	<xacro:kuka_kr16_2  prefix="kr16_">
 	</xacro:kuka_kr16_2>
-	<xacro:axia80_adapter_robotside_flange  parent_link="${prefix}tool0">
+	<xacro:axia80_adapter_robotside_flange  parent_link="kr16_tool0">
 		<origin xyz="0 0 0" rpy="0 0 ${pi/2}" />
 	</xacro:axia80_adapter_robotside_flange>
@@ -15,5 +15,5 @@
 		<origin xyz="0 0 0" rpy="0 0 0" />
 	</xacro:ati_axia80>
-	<xacro:axia80_adapter_toolside_sensor  parent_link="${prefix}toolside">
+	<xacro:axia80_adapter_toolside_sensor  parent_link="ati_axia80_toolside">
 		<origin xyz="0 0 0" rpy="0 0 0" />
 	</xacro:axia80_adapter_toolside_sensor>
@@ -24,5 +24,5 @@
 	<joint name="table_joint" type="fixed">
 		<parent link="table_big" />
-		<child link="${prefix}base_link" />
+		<child link="kr16_base_link" />
 		<origin xyz="0.858 0.863 -0.405" rpy="0 0 ${-3/4*pi}" />
 	</joint>
