Commit message: fix tag closure generated

File: examples/generated/PiTasc/kr16_2_macro.xacro (robot description, xacro)
@@ -14,5 +14,5 @@
 			</collision>
 			<inertial>
-				<mass value="2.0">
+				<mass value="2.0" />
 				<origin xyz="0 0 0" rpy="0 0 0" />
 				<inertia ixx="0.01" ixy="0.0" ixz="0.0"
@@ -33,5 +33,5 @@
 			</collision>
 			<inertial>
-				<mass value="2.0">
+				<mass value="2.0" />
 				<origin xyz="0 0 0" rpy="0 0 0" />
 				<inertia ixx="0.01" ixy="0.0" ixz="0.0"
@@ -52,5 +52,5 @@
 			</collision>
 			<inertial>
-				<mass value="2.0">
+				<mass value="2.0" />
 				<origin xyz="0 0 0" rpy="0 0 0" />
 				<inertia ixx="0.01" ixy="0.0" ixz="0.0"
@@ -71,5 +71,5 @@
 			</collision>
 			<inertial>
-				<mass value="2.0">
+				<mass value="2.0" />
 				<origin xyz="0 0 0" rpy="0 0 0" />
 				<inertia ixx="0.01" ixy="0.0" ixz="0.0"
@@ -90,5 +90,5 @@
 			</collision>
 			<inertial>
-				<mass value="2.0">
+				<mass value="2.0" />
 				<origin xyz="0 0 0" rpy="0 0 0" />
 				<inertia ixx="0.01" ixy="0.0" ixz="0.0"
@@ -109,5 +109,5 @@
 			</collision>
 			<inertial>
-				<mass value="2.0">
+				<mass value="2.0" />
 				<origin xyz="0 0 0" rpy="0 0 0" />
 				<inertia ixx="0.01" ixy="0.0" ixz="0.0"
@@ -128,5 +128,5 @@
 			</collision>
 			<inertial>
-				<mass value="2.0">
+				<mass value="2.0" />
 				<origin xyz="0 0 0" rpy="0 0 0" />
 				<inertia ixx="0.01" ixy="0.0" ixz="0.0"
@@ -145,5 +145,5 @@
 			<child link="${prefix}link_1" />
 			<origin xyz="0 0 0.675" rpy="0 0 0" />
-			<axis xyz="0 0 -1">
+			<axis xyz="0 0 -1" />
 		</joint>
 		<joint name="${prefix}joint_a2" type="revolute">
@@ -151,5 +151,5 @@
 			<child link="${prefix}link_2" />
 			<origin xyz="0.26 0 0" rpy="0 0 0" />
-			<axis xyz="0 1 0">
+			<axis xyz="0 1 0" />
 		</joint>
 		<joint name="${prefix}joint_a3" type="revolute">
@@ -157,5 +157,5 @@
 			<child link="${prefix}link_3" />
 			<origin xyz="0.68 0 0" rpy="0 0 0" />
-			<axis xyz="0 1 0">
+			<axis xyz="0 1 0" />
 		</joint>
 		<joint name="${prefix}joint_a4" type="revolute">
@@ -163,5 +163,5 @@
 			<child link="${prefix}link_4" />
 			<origin xyz="0.67 0 -0.035" rpy="0 0 0" />
-			<axis xyz="-1 0 0">
+			<axis xyz="-1 0 0" />
 		</joint>
 		<joint name="${prefix}joint_a5" type="revolute">
@@ -169,5 +169,5 @@
 			<child link="${prefix}link_5" />
 			<origin xyz="0 0 0" rpy="0 0 0" />
-			<axis xyz="0 1 0">
+			<axis xyz="0 1 0" />
 		</joint>
 		<joint name="${prefix}joint_a6" type="revolute">
@@ -180,5 +180,5 @@
 			<child link="${prefix}flange" />
 			<origin xyz="0.158 0 0" rpy="0 0 0" />
-			<axis xyz="-1 0 0">
+			<axis xyz="-1 0 0" />
 		</joint>
 		<joint name="${prefix}base_link_base" type="revolute">

Commit message: re-generated files from example models

File: examples/generated/PiTasc/kr16_2_macro.xacro (robot description, xacro)
@@ -142,6 +142,6 @@
 		</link>
 		<joint name="${prefix}joint_a1" type="revolute">
-			<parent link="${prefix}base_link" />
-			<child link="${prefix}link_1" />
+			<parent link="kr16_base_link" />
+			<child link="kr16_link_1" />
 			<origin xyz="0 0 0.675" rpy="0 0 0" />
 			<axis xyz="0 0 -1" />
@@ -149,6 +149,6 @@
 		</joint>
 		<joint name="${prefix}joint_a2" type="revolute">
-			<parent link="${prefix}link_1" />
-			<child link="${prefix}link_2" />
+			<parent link="kr16_link_1" />
+			<child link="kr16_link_2" />
 			<origin xyz="0.26 0 0" rpy="0 0 0" />
 			<axis xyz="0 1 0" />
@@ -156,6 +156,6 @@
 		</joint>
 		<joint name="${prefix}joint_a3" type="revolute">
-			<parent link="${prefix}link_2" />
-			<child link="${prefix}link_3" />
+			<parent link="kr16_link_2" />
+			<child link="kr16_link_3" />
 			<origin xyz="0.68 0 0" rpy="0 0 0" />
 			<axis xyz="0 1 0" />
@@ -163,6 +163,6 @@
 		</joint>
 		<joint name="${prefix}joint_a4" type="revolute">
-			<parent link="${prefix}link_3" />
-			<child link="${prefix}link_4" />
+			<parent link="kr16_link_3" />
+			<child link="kr16_link_4" />
 			<origin xyz="0.67 0 -0.035" rpy="0 0 0" />
 			<axis xyz="-1 0 0" />
@@ -170,6 +170,6 @@
 		</joint>
 		<joint name="${prefix}joint_a5" type="revolute">
-			<parent link="${prefix}link_4" />
-			<child link="${prefix}link_5" />
+			<parent link="kr16_link_4" />
+			<child link="kr16_link_5" />
 			<origin xyz="0 0 0" rpy="0 0 0" />
 			<axis xyz="0 1 0" />
@@ -177,23 +177,23 @@
 		</joint>
 		<joint name="${prefix}joint_a6" type="revolute">
-			<parent link="${prefix}link_5" />
-			<child link="${prefix}link_6" />
+			<parent link="kr16_link_5" />
+			<child link="kr16_link_6" />
 			<origin xyz="0 0 0.675" rpy="0 0 0" />
 			<limit effort="0" lower="${radians(-350)}" upper="${radians(350)}" velocity="${radians(615)}" />
 		</joint>
 		<joint name="${prefix}joint_a6_flange" type="revolute">
-			<parent link="${prefix}link_6" />
-			<child link="${prefix}flange" />
+			<parent link="kr16_link_6" />
+			<child link="kr16_flange" />
 			<origin xyz="0.158 0 0" rpy="0 0 0" />
 			<axis xyz="-1 0 0" />
 		</joint>
 		<joint name="${prefix}base_link_base" type="revolute">
-			<parent link="${prefix}base_link" />
-			<child link="${prefix}base" />
+			<parent link="kr16_base_link" />
+			<child link="kr16_base" />
 			<origin xyz="0 0 0.675" rpy="0 0 0" />
 		</joint>
 		<joint name="${prefix}flange_tool0" type="revolute">
-			<parent link="${prefix}flange" />
-			<child link="${prefix}tool0" />
+			<parent link="kr16_flange" />
+			<child link="kr16_tool0" />
 			<origin xyz="0 0 0" rpy="0 ${radians(90)} 0" />
 		</joint>
