Commit message: added parameter types to models

File: examples/PiTasc/ati_axia80.xacro (robot description, xacro)
@@ -3,7 +3,7 @@
 		Macro { name ati_axia80
 			parameter {
-				Parameter parent_link {},
-				Parameter prefix {},
-				Parameter origin_joint {} }
+				Parameter parent_link { type LinkRef},
+				Parameter prefix { type String },
+				Parameter origin_joint { type Pose } }
 			body Body {
 				link {

File: examples/PiTasc/axia80_adapter_plates.xacro (robot description, xacro)
@@ -3,6 +3,6 @@
 		Macro { name axia80_adapter_robotside_flange
 			parameter {
-				Parameter parent_link { },
-				Parameter origin_joint { } }
+				Parameter parent_link { type LinkRef },
+				Parameter origin_joint { type Pose } }
 			body Body {
 				link {
@@ -22,6 +22,6 @@
 		Macro { name axia80_adapter_robotside_sensor
 			parameter {
-				Parameter parent_link {},
-				Parameter origin_joint {} }
+				Parameter parent_link { type LinkRef },
+				Parameter origin_joint {type Pose } }
 			body Body {
 				link {
@@ -46,6 +46,6 @@
 		Macro { name axia80_adapter_toolside_sensor
 			parameter {
-				Parameter parent_link {},
-				Parameter origin_joint {} }
+				Parameter parent_link { type LinkRef },
+				Parameter origin_joint { type Pose } }
 			body Body {
 				link {

File: examples/PiTasc/kr16_2_macro.xacro (robot description, xacro)
@@ -3,5 +3,5 @@
 		Macro { name kuka_kr16_2
 			parameter {
-				Parameter prefix {} }
+				Parameter prefix { type String } }
 			body Body {
 				link {

File: examples/generated/PiTasc/ati_axia80.xacro (robot description, xacro)
@@ -1,5 +1,5 @@
 <?xml version="1.0"?>
 <robot xmlns:xacro="http://wiki.ros.org/xacro" name="ati_axia80" >
-	<xacro:macro name="ati_axia80" params="parent_link prefix origin_joint ">
+	<xacro:macro name="ati_axia80" params="parent_link prefix *origin_joint ">
 		<link name="${prefix}robotside" >
 			<visual>
@@ -15,15 +15,15 @@
 		<joint name="${prefix}robotside_joint" type="fixed">
 			<parent link="${parent_link}" />
-			<child link="ati_axia80_robotside" />
+			<child link="${prefix}robotside" />
 			<xacro:insert_block name="origin_joint"/>
 		</joint>
 		<joint name="${prefix}toolside_joint" type="fixed">
-			<parent link="ati_axia80_robotside" />
-			<child link="ati_axia80_toolside" />
+			<parent link="${prefix}robotside" />
+			<child link="${prefix}toolside" />
 			<origin xyz="0 0 0" rpy="0 0 0.0254" />
 		</joint>
 		<joint name="${prefix}measurement_joint" type="fixed">
-			<parent link="ati_axia80_toolside" />
-			<child link="ati_axia80_force_sensor_frame" />
+			<parent link="${prefix}toolside" />
+			<child link="${prefix}force_sensor_frame" />
 			<origin xyz="0 0 0" rpy="0 0 0" />
 		</joint>

File: examples/generated/PiTasc/axia80_adapter_plates.xacro (robot description, xacro)
@@ -1,5 +1,5 @@
 <?xml version="1.0"?>
 <robot xmlns:xacro="http://wiki.ros.org/xacro" name="axia80_adapter_plates" >
-	<xacro:macro name="axia80_adapter_robotside_flange" params="parent_link origin_joint ">
+	<xacro:macro name="axia80_adapter_robotside_flange" params="parent_link *origin_joint ">
 		<link name="axia80_adapter_robotside_flange" >
 		</link>
@@ -17,5 +17,5 @@
 		</joint>
 	</xacro:macro>
-	<xacro:macro name="axia80_adapter_robotside_sensor" params="parent_link origin_joint ">
+	<xacro:macro name="axia80_adapter_robotside_sensor" params="parent_link *origin_joint ">
 		<link name="axia80_adapter_robotside_changer_sensor" >
 			<visual>
@@ -38,5 +38,5 @@
 		</joint>
 	</xacro:macro>
-	<xacro:macro name="axia80_adapter_toolside_sensor" params="parent_link origin_joint ">
+	<xacro:macro name="axia80_adapter_toolside_sensor" params="parent_link *origin_joint ">
 		<link name="axia80_adapter_toolside_sensor" >
 		</link>
