Commit message: add limits to revolute joints

File: examples/PiTasc/kr16_2_macro.xacro (robot description, xacro)
@@ -106,5 +106,6 @@
 						child "prefixlink_1"
 						origin Pose { rpy "0 0 0" xyz "0 0 0.675" }
-						axis Vector3 { xyz "0 0 -1" } },
+						axis Vector3 { xyz "0 0 -1" }
+						limit Limit { effort "0" lower "${radians(-185)}" upper "${radians(185)}" velocity "${radians(156)}" } },
 					 Joint { name "prefix"joint_a2
 						type revolute
@@ -112,5 +113,6 @@
 						child "prefixlink_2"
 						origin Pose { rpy "0 0 0" xyz "0.26 0 0" }
-						axis Vector3 { xyz "0 1 0" } },
+						axis Vector3 { xyz "0 1 0" }
+						limit Limit { effort "0" lower "${radians(-155)}" upper "${radians(35)}" velocity "${radians(156)}" } },
 					Joint { name "prefix"joint_a3
 						type revolute
@@ -118,5 +120,6 @@
 						child "prefixlink_3"
 						origin Pose { rpy "0 0 0" xyz "0.68 0 0" }
-						axis Vector3 { xyz "0 1 0" } },
+						axis Vector3 { xyz "0 1 0" }
+						limit Limit { effort "0" lower "${radians(-130)}" upper "${radians(154)}" velocity "${radians(156)}" } },
 					Joint { name "prefix"joint_a4
 						type revolute
@@ -124,5 +127,6 @@
 						child "prefixlink_4"
 						origin Pose { rpy "0 0 0" xyz "0.67 0 -0.035" }
-						axis Vector3 { xyz "-1 0 0" } },
+						axis Vector3 { xyz "-1 0 0" }
+						limit Limit { effort "0" lower "${radians(-350)}" upper "${radians(350)}" velocity "${radians(330)}" } },
 					Joint { name "prefix"joint_a5
 						type revolute
@@ -130,10 +134,12 @@
 						child "prefixlink_5"
 						origin Pose { rpy "0 0 0" xyz "0 0 0" }
-						axis Vector3 { xyz "0 1 0" } },
+						axis Vector3 { xyz "0 1 0" }
+						limit Limit { effort "0" lower "${radians(-130)}" upper "${radians(130)}" velocity "${radians(330)}" } },
 					Joint { name "prefix"joint_a6
 						type revolute
 						parent "prefixlink_5"
 						child "prefixlink_6"
-						origin Pose { rpy "0 0 0" xyz "0 0 0.675" } },
+						origin Pose { rpy "0 0 0" xyz "0 0 0.675" }
+						limit Limit { effort "0" lower "${radians(-350)}" upper "${radians(350)}" velocity "${radians(615)}" } },
 					Joint { name "prefix"joint_a6_flange
 						type revolute

File: examples/generated/PiTasc/ati_axia80.xacro (robot description, xacro)
@@ -15,15 +15,15 @@
 		<joint name="${prefix}robotside_joint" type="fixed">
 			<parent link="${parent_link}" />
-			<child link="${prefix}robotside" />
+			<child link="ati_axia80_robotside" />
 			<xacro:insert_block name="origin_joint"/>
 		</joint>
 		<joint name="${prefix}toolside_joint" type="fixed">
-			<parent link="${prefix}robotside" />
-			<child link="${prefix}toolside" />
+			<parent link="ati_axia80_robotside" />
+			<child link="ati_axia80_toolside" />
 			<origin xyz="0 0 0" rpy="0 0 0.0254" />
 		</joint>
 		<joint name="${prefix}measurement_joint" type="fixed">
-			<parent link="${prefix}toolside" />
-			<child link="${prefix}force_sensor_frame" />
+			<parent link="ati_axia80_toolside" />
+			<child link="ati_axia80_force_sensor_frame" />
 			<origin xyz="0 0 0" rpy="0 0 0" />
 		</joint>

File: examples/generated/PiTasc/kr16_2_macro.xacro (robot description, xacro)
@@ -146,4 +146,5 @@
 			<origin xyz="0 0 0.675" rpy="0 0 0" />
 			<axis xyz="0 0 -1" />
+			<limit effort="0" lower="${radians(-185)}" upper="${radians(185)}" velocity="${radians(156)}" />
 		</joint>
 		<joint name="${prefix}joint_a2" type="revolute">
@@ -152,4 +153,5 @@
 			<origin xyz="0.26 0 0" rpy="0 0 0" />
 			<axis xyz="0 1 0" />
+			<limit effort="0" lower="${radians(-155)}" upper="${radians(35)}" velocity="${radians(156)}" />
 		</joint>
 		<joint name="${prefix}joint_a3" type="revolute">
@@ -158,4 +160,5 @@
 			<origin xyz="0.68 0 0" rpy="0 0 0" />
 			<axis xyz="0 1 0" />
+			<limit effort="0" lower="${radians(-130)}" upper="${radians(154)}" velocity="${radians(156)}" />
 		</joint>
 		<joint name="${prefix}joint_a4" type="revolute">
@@ -164,4 +167,5 @@
 			<origin xyz="0.67 0 -0.035" rpy="0 0 0" />
 			<axis xyz="-1 0 0" />
+			<limit effort="0" lower="${radians(-350)}" upper="${radians(350)}" velocity="${radians(330)}" />
 		</joint>
 		<joint name="${prefix}joint_a5" type="revolute">
@@ -170,4 +174,5 @@
 			<origin xyz="0 0 0" rpy="0 0 0" />
 			<axis xyz="0 1 0" />
+			<limit effort="0" lower="${radians(-130)}" upper="${radians(130)}" velocity="${radians(330)}" />
 		</joint>
 		<joint name="${prefix}joint_a6" type="revolute">
@@ -175,4 +180,5 @@
 			<child link="${prefix}link_6" />
 			<origin xyz="0 0 0.675" rpy="0 0 0" />
+			<limit effort="0" lower="${radians(-350)}" upper="${radians(350)}" velocity="${radians(615)}" />
 		</joint>
 		<joint name="${prefix}joint_a6_flange" type="revolute">
